Commit message: Adding friction and damping to the grippers joints

File: robotiq_description/urdf/robotiq_2f_140.xacro (robot description, xacro)
@@ -151,4 +151,5 @@
       <axis xyz="-1 0 0" />
       <limit lower="0" upper="0.7" velocity="2.0" effort="1000" />
+      <dynamics damping="0.5" friction="1" />
     </joint>
     <xacro:finger_joints prefix="${prefix}" fingerprefix="left" reflect="1.0"/>
@@ -161,4 +162,5 @@
       <axis xyz="1 0 0" />
       <limit lower="-0.725" upper="0.725" velocity="2.0" effort="1000" />
+      <dynamics damping="0.5" friction="1" />
     <mimic joint="${prefix}finger_joint" multiplier="-1" offset="0" />
     </joint>
@@ -180,4 +182,5 @@
       <axis xyz="1 0 0" />
       <limit lower="-0.8757" upper="0.8757" velocity="2.0" effort="1000" />
+      <dynamics damping="0.5" friction="1" />
       <mimic joint="${prefix}finger_joint" multiplier="-1" offset="0" />
     </joint>
@@ -190,4 +193,5 @@
       <axis xyz="1 0 0" />
       <limit lower="-0.8757" upper="0.8757" velocity="2.0" effort="1000" />
+      <dynamics damping="0.5" friction="1" />
       <mimic joint="${prefix}finger_joint" multiplier="1" offset="0" />
     </joint>

File: robotiq_description/urdf/robotiq_2f_85_macro.urdf.xacro (robot description, xacro)
@@ -228,4 +228,5 @@
             <origin xyz="0.03060114 0.0 0.05490452" rpy="0 0 0" />
             <limit lower="0.0" upper="0.8" velocity="0.5" effort="50" />
+            <dynamics damping="0.05" friction="0.1" />
         </joint>
         <joint name="${prefix}robotiq_85_right_knuckle_joint" type="revolute">
@@ -235,4 +236,5 @@
             <origin xyz="-0.03060114 0.0 0.05490452" rpy="0 0 0" />
             <limit lower="-0.8" upper="0.0" velocity="0.5" effort="50" />
+            <dynamics damping="0.05" friction="0.1" />
             <mimic joint="${prefix}robotiq_85_left_knuckle_joint" multiplier="-1" />
         </joint>
