Commit message: Modified the friction and damping coefficients for 2f_85

File: robotiq_description/urdf/robotiq_2f_85_macro.urdf.xacro (robot description, xacro)
@@ -228,5 +228,5 @@
             <origin xyz="0.03060114 0.0 0.05490452" rpy="0 0 0" />
             <limit lower="0.0" upper="0.8" velocity="0.5" effort="50" />
-            <dynamics damping="0.05" friction="0.1" />
+            <dynamics damping="0.5" friction="1" />
         </joint>
         <joint name="${prefix}robotiq_85_right_knuckle_joint" type="revolute">
@@ -236,5 +236,5 @@
             <origin xyz="-0.03060114 0.0 0.05490452" rpy="0 0 0" />
             <limit lower="-0.8" upper="0.0" velocity="0.5" effort="50" />
-            <dynamics damping="0.05" friction="0.1" />
+            <dynamics damping="0.5" friction="1" />
             <mimic joint="${prefix}robotiq_85_left_knuckle_joint" multiplier="-1" />
         </joint>
